Commit message: ++ FF scripts

File: plate.urdf (robot description, URDF)
Before this commit: robot plate, 3 links, 2 joints
Links:
- link plate_link: geometry collision box size=0.40 0.50 0.0052; visual box size=0.40 0.40 0.0052
- link small_link: mass None -> 0

Commit message: ++ CTRNN

File: plate.urdf (robot description, URDF)
Before this commit: robot plate, 3 links, 2 joints
Links:
- link plate_link: geometry collision box size=0.40 0.40 0.0052; visual box size=0.40 0.40 0.0052
